File: Kicad/FireFlyLid/FireFlyLid.sch (KiCad schematic (older format))
At the start: 52 parts, among them J1 HEADER_4, J2 HEADER_1, J3 HEADER_1, SW1 SW_SPDT, U1 MSP430G2553IPW28, U2 MAXIM_MAX44009, X1 32K

Commit message: New layout with off board battery and local vreg to 3.0 V
Parts:
- added C3: 1uF, ~, symbol CAP
- added C4: 470pF, ~, symbol CAP
- added VDET1: VDETECTOR_3PINS-SOT-223, dp_devices-SOT-223, symbol VDETECTOR_3PINS-SOT-223
- added VREG1: VREG_5PINS-SOT-23-5, dp_devices-SOT-23-5, symbol VREG_5PINS-SOT-23-5
Connections:
- net labels added: PROG_VCC
- wire segments 11 -> 18
- no-connect marks 1 -> 0
Other:
- note added: "POWER MANAGEMENT"
- note removed: "BATTERY POWER"
- moved on the sheet: BAT1, J1, J2, J3, LD1, LD10, LD11, LD12, LD13, LD14, LD15, LD16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

Commit message: mid work
Other:
- note added: "Change P3.7 for interrupt to use P1 or P2"
Changed lines of the file:
@@
 Sheet 1 1
 Title ""
-Date "21 sep 2014"
+Date "15 feb 2015"
 Rev ""
 Comp ""
@@
 Wire Wire Line
 	2350 6000 2350 6100
+Text Notes 8250 3050 0    60   ~ 0
+Change P3.7 for interrupt to use P1 or P2
 $EndSCHEMATC
